File: PCB/night-activated-switch.brd (EAGLE design)
At the start: 33 x 20 mm, 13 parts, among them Q1 2N7002

Commit message: Update voltage divider values.
Parts:
- R5: value 12K -> 5K
- R6: value 10K -> 3.3K
Changed lines of the file:
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@@
 </layers>
 <board>
-<fusionsync huburn="a.cGVyc29uYWw6dWUyYmRlZGJl" projecturn="a.cGVyc29uYWw6dWUyYmRlZGJlIzIwMTgwNTA0MTMwNTkwMzU2" f3durn="urn:adsk.wipprod:dm.lineage:vwfqz0IPQgaWsHL0F2eGuQ" pcbguid="7f8044df-318b-45b2-bb71-742f6d91b34a" lastpulledtime="" lastsyncedchangeguid="" latestrevisionid="0b2277a9-b629-4486-bf19-4959c4c3a7e3" lastsyncedrevisionid="0b2277a9-b629-4486-bf19-4959c4c3a7e3" lastboardhashguid="9a09c57e-ac53-11eb-4370-254c3b2cf7b0" lastpushedtime="2022-04-12T03:25:34Z" linktopcb3d="true"/>
+<fusionsync huburn="a.cGVyc29uYWw6dWUyYmRlZGJl" projecturn="a.cGVyc29uYWw6dWUyYmRlZGJlIzIwMTgwNTA0MTMwNTkwMzU2" f3durn="urn:adsk.wipprod:dm.lineage:vwfqz0IPQgaWsHL0F2eGuQ" pcbguid="" lastpulledtime="" lastsyncedchangeguid="" latestrevisionid="0b2277a9-b629-4486-bf19-4959c4c3a7e3" lastsyncedrevisionid="0b2277a9-b629-4486-bf19-4959c4c3a7e3" lastboardhashguid="9a09c57e-ac53-11eb-4370-254c3b2cf7b0" lastpushedtime="2022-04-12T03:25:34Z" linktopcb3d="true"/>
 <plain>
 <wire x1="0" y1="0" x2="33" y2="0" width="0" layer="20"/>
@@
 <attribute name="VALUE" x="22" y="2.5" size="0.2" layer="28" rot="MR0" align="center"/>
 </element>
-<element name="R5" library="rlc" library_urn="urn:adsk.eagle:library:4192893" package="0603-RES" package3d_urn="urn:adsk.eagle:package:4193040/2" value="12K" x="22" y="7.5" smashed="yes" rot="MR180">
+<element name="R5" library="rlc" library_urn="urn:adsk.eagle:library:4192893" package="0603-RES" package3d_urn="urn:adsk.eagle:package:4193040/2" value="5K" x="22" y="7.5" smashed="yes" rot="MR180">
 <attribute name="NAME" x="20.5" y="7.5" size="0.8128" layer="26" font="vector" ratio="15" rot="MR0" align="center-left"/>
 <attribute name="VALUE" x="22" y="7.7" size="0.2" layer="28" rot="MR180" align="center"/>
 </element>
-<element name="R6" library="rlc" library_urn="urn:adsk.eagle:library:4192893" package="0603-RES" package3d_urn="urn:adsk.eagle:package:4193040/2" value="10K" x="22" y="8.7" smashed="yes" rot="MR0">
+<element name="R6" library="rlc" library_urn="urn:adsk.eagle:library:4192893" package="0603-RES" package3d_urn="urn:adsk.eagle:package:4193040/2" value="3.3K" x="22" y="8.7" smashed="yes" rot="MR0">
 <attribute name="NAME" x="20.5" y="8.7" size="0.8128" layer="26" font="vector" ratio="15" rot="MR0" align="center-left"/>
 <attribute name="VALUE" x="22" y="8.5" size="0.2" layer="28" rot="MR0" align="center"/>
